File: calcifer_devboard.kicad_pcb (KiCad board)
At the start: 2 copper layers, 58.2 x 70.9 mm, 34 parts, among them J1 USB_C_Receptacle_USB2.0_14P, J2 Conn_01x03, J3 Conn_01x20, J4 Conn_01x20, SW1 SW_Push, U1 RP2040, U2 NCP1117-3.3_SOT223, U3 W25Q128JVS, Y1 23 MHz

Commit message: retraced everything and finished readme
Parts:
- moved C6 15.3 mm to (137.8, 98.5)
- moved C8 12.2 mm to (132.0, 103.8), turned to -90 degrees
- moved C11 11.5 mm to (131.0, 103.8), turned to -90 degrees
- moved C10 11.5 mm to (134.0, 91.5), turned to 90 degrees
- moved C3 9.76 mm to (133.5, 90.0), turned to 0 degrees
- moved C12 3.63 mm to (129.5, 91.5), turned to 90 degrees
- moved C7 3.15 mm to (133.0, 91.5)
- moved C4 3.00 mm to (127.5, 94.0)
- moved C16 1.99 mm to (130.0, 104.8), turned to 90 degrees
- moved U3 1.97 mm to (134.9, 85.0)
- moved C17 1.96 mm to (130.9, 81.9)
- moved R4 1.96 mm to (138.8, 81.9)
- moved R6 1.78 mm to (131.7, 90.5)
- moved R7 1.78 mm to (130.5, 90.5)
- moved C2 1.78 mm to (128.0, 93.0)
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Routing:
- net GND: track 52.8 -> 37.2 mm, vias 11 -> 16
- net USB_D-: track 38.1 -> 46.6 mm
- net USB_D+: track 38.1 -> 46.6 mm
- net +3V3: track 124.6 -> 117.5 mm, vias 3 -> 6
- net +1V1: track 20.0 -> 26.6 mm, vias 6 -> 3
- net GPIO0: track 41.7 -> 36.7 mm
- net GPIO16: track 43.4 -> 48.2 mm
- net QSPI_SCLK: track 8.83 -> 13.4 mm, vias 0 -> 2
- net QSPI_SD0: track 6.16 -> 10.7 mm, vias 0 -> 2
- net GPIO17: track 41.8 -> 46.3 mm
- net GPIO18: track 38.4 -> 42.6 mm
- net SWD: track 30.6 -> 34.8 mm
- net GPIO19: track 38.1 -> 42.2 mm
- net GPIO20: track 36.7 -> 40.8 mm
- net QSPI_SD3: track 10.3 -> 14.3 mm, vias 0 -> 2
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
Commit message: Silkscreen update and complete README
Other:
- board text added: "SWCLK"
- board text added: "SWD"
Changed lines of the file:
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@@
 		(tags "resistor")
 		(property "Reference" "R5"
-			(at 0 1.17 0)
+			(at 0.0125 1.065 0)
 			(layer "B.SilkS")
 			(effects
 				(font
-					(size 1 1)
-					(thickness 0.15)
+					(size 0.254 0.254)
+					(thickness 0.0635)
 				)
 				(justify mirror)
@@
 		(tags "capacitor")
 		(property "Reference" "C8"
-			(at 0 1.16 90)
+			(at -1.26 0 180)
 			(layer "B.SilkS")
 			(effects
 				(font
-					(size 1 1)
-					(thickness 0.15)
+					(size 0.254 0.254)
+					(thickness 0.0635)
 				)
 				(justify mirror)
@@
 		(tags "capacitor")
 		(property "Reference" "C3"
-			(at 0 1.16 0)
+			(at 0 -0.75 0)
 			(layer "B.SilkS")
 			(effects
 				(font
-					(size 1 1)
-					(thickness 0.15)
+					(size 0.254 0.254)
+					(thickness 0.0635)
 				)
 				(justify mirror)
@@
 		(tags "capacitor")
 		(property "Reference" "C4"
-			(at 0 1.16 0)
+			(at 1.5 0 0)
 			(layer "B.SilkS")
 			(effects
 				(font
-					(size 1 1)
-					(thickness 0.15)
+					(size 0.254 0.254)
+					(thickness 0.0635)
 				)
 				(justify mirror)
@@
 		(tags "capacitor")
 		(property "Reference" "C14"
-			(at 0 1.16 135)
+			(at 1.626346 -0.141421 135)
 			(layer "B.SilkS")
 			(effects
 				(font
-					(size 1 1)
-					(thickness 0.15)
+					(size 0.254 0.254)
+					(thickness 0.0635)
 				)
 				(justify mirror)
@@
 		(tags "QFN NoLead")
 		(property "Reference" "U1"
-			(at -0.2 4.73 0)
+			(at 1.2625 5 0)
 			(layer "B.SilkS")
 			(effects
@@
 		(tags "capacitor")
 		(property "Reference" "C11"
-			(at 0 1.16 90)
+			(at -1.26 0 180)
 			(layer "B.SilkS")
 			(effects
 				(font
-					(size 1 1)
-					(thickness 0.15)
+					(size 0.254 0.254)
+					(thickness 0.0635)
 				)
 				(justify mirror)
@@
 		(tags "capacitor")
 		(property "Reference" "C17"
-			(at 0 1.16 0)
+			(at 1.4125 -0.1 0)
 			(layer "B.SilkS")
 			(effects
 				(font
-					(size 1 1)
-					(thickness 0.15)
+					(size 0.254 0.254)
+					(thickness 0.0635)
 				)
 				(justify mirror)
@@
 		(tags "resistor")
 		(property "Reference" "R7"
-			(at 0 1.17 90)
+			(at -1.2565 -0.0375 180)
 			(layer "B.SilkS")
 			(effects
 				(font
-					(size 1 1)
-					(thickness 0.15)
+					(size 0.254 0.254)
+					(thickness 0.0635)
 				)
 				(justify mirror)
@@
 		(tags "capacitor")
 		(property "Reference" "C6"
-			(at 0 1.16 0)
+			(at 0 -1 0)
 			(layer "B.SilkS")
 			(effects
 				(font
-					(size 1 1)
-					(thickness 0.15)
+					(size 0.254 0.254)
+					(thickness 0.0635)
 				)
 				(justify mirror)
@@
 		(tags "capacitor")
 		(property "Reference" "C10"
-			(at 0 1.16 90)
+			(at -1.23 0 180)
 			(layer "B.SilkS")
 			(effects
 				(font
-					(size 1 1)
-					(thickness 0.15)
+					(size 0.254 0.254)
+					(thickness 0.0635)
 				)
 				(justify mirror)
@@
 		(tags "capacitor")
 		(property "Reference" "C15"
-			(at 0 1.16 90)
+			(at 1.26 0 180)
 			(layer "B.SilkS")
 			(effects
 				(font
-					(size 1 1)
-					(thickness 0.15)
+					(size 0.254 0.254)
+					(thickness 0.0635)
 				)
 				(justify mirror)
@@
 		(tags "capacitor")
 		(property "Reference" "C12"
-			(at 0 1.16 90)
+			(at 1.5 0 180)
 			(layer "B.SilkS")
 			(effects
 				(font
-					(size 1 1)
-					(thickness 0.15)
+					(size 0.254 0.254)
+					(thickness 0.0635)
 				)
 				(justify mirror)
@@
 		(tags "capacitor")
 		(property "Reference" "C2"
-			(at 0 1.16 0)
+			(at 0.5 0.75 0)
 			(layer "B.SilkS")
 			(effects
 				(font
-					(size 1 1)
-					(thickness 0.15)
+					(size 0.254 0.254)
+					(thickness 0.0635)
 				)
 				(justify mirror)
@@
 		(tags "resistor")
 		(property "Reference" "R2"
-			(at 0 1.17 45)
+			(at 0.070711 0.777817 45)
 			(layer "B.SilkS")
 			(effects
 				(font
-					(size 1 1)
-					(thickness 0.15)
+					(size 0.254 0.254)
+					(thickness 0.0635)
 				)
 				(justify mirror)
@@
 		(tags "capacitor")
 		(property "Reference" "C16"
-			(at 0 1.16 90)
+			(at 1.25 0 180)
 			(layer "B.SilkS")
 			(effects
 				(font
-					(size 1 1)
-					(thickness 0.15)
+					(size 0.254 0.254)
+					(thickness 0.0635)
 				)
 				(justify mirror)
@@
 		(tags "resistor")
 		(property "Reference" "R3"
-			(at 0 1.17 90)
+			(at 1.26 0 180)
 			(layer "B.SilkS")
 			(effects
 				(font
-					(size 1 1)
-					(thickness 0.15)
+					(size 0.254 0.254)
+					(thickness 0.0635)
 				)
 				(justify mirror)
@@
 		(tags "usb usb-c 2.0 pd")
 		(property "Reference" "J1"
-			(at 0 5.645 135)
+			(at -0.106066 6.322921 135)
 			(layer "B.SilkS")
 			(effects
@@
 		(tags "capacitor")
 		(property "Reference" "C5"
-			(at 0 1.16 0)
+			(at 0.02 1 0)
 			(layer "B.SilkS")
 			(effects
 				(font
-					(size 1 1)
-					(thickness 0.15)
+					(size 0.254 0.254)
+					(thickness 0.0635)
 				)
 				(justify mirror)
@@
 		(tags "capacitor")
 		(property "Reference" "C1"
-			(at 0 1.16 90)
+			(at 0.73 -1 180)
 			(layer "B.SilkS")
 			(effects
 				(font
-					(size 1 1)
-					(thickness 0.15)
+					(size 0.254 0.254)
+					(thickness 0.0635)
 				)
 				(justify mirror)
@@
 		(tags "resistor")
 		(property "Reference" "R6"
-			(at 0 1.17 90)
+			(at -1.2565 -0.0875 180)
 			(layer "B.SilkS")
 			(effects
 				(font
-					(size 1 1)
-					(thickness 0.15)
+					(size 0.254 0.254)
+					(thickness 0.0635)
 				)
 				(justify mirror)
@@
 		(tags "resistor")
 		(property "Reference" "R4"
-			(at 0 1.17 0)
+			(at 1.4375 0.1 0)
 			(layer "B.SilkS")
 			(effects
 				(font
-					(size 1 1)
-					(thickness 0.15)
+					(size 0.254 0.254)
+					(thickness 0.0635)
 				)
 				(justify mirror)
@@
 		(tags "resistor")
 		(property "Reference" "R1"
-			(at 0 1.17 135)
+			(at -1.626346 0 135)
 			(layer "B.SilkS")
 			(effects
 				(font
-					(size 1 1)
-					(thickness 0.15)
+					(size 0.254 0.254)
+					(thickness 0.0635)
 				)
 				(justify mirror)
@@
 		(tags "capacitor")
 		(property "Reference" "C9"
-			(at 0 1.16 0)
+			(at 0.02 -1 0)
 			(layer "B.SilkS")
 			(effects
 				(font
-					(size 1 1)
-					(thickness 0.15)
+					(size 0.254 0.254)
+					(thickness 0.0635)
 				)
 				(justify mirror)
@@
 			(effects
 				(font
-					(size 1 1)
-					(thickness 0.15)
+					(size 0.254 0.254)
+					(thickness 0.0635)
 				)
 				(justify mirror)
@@
 		(tags "capacitor")
 		(property "Reference" "C7"
-			(at 0 1.16 90)
+			(at -1.25 0 180)
 			(layer "B.SilkS")
 			(effects
 				(font
-					(size 1 1)
-					(thickness 0.15)
+					(size 0.254 0.254)
+					(thickness 0.0635)
 				)
 				(justify mirror)
@@
 		)
 	)
+	(gr_text "SWD"
+		(at 150.5 98.25 0)
+		(layer "B.SilkS")
+		(effects
+			(font
+				(size 0.762 0.762)
+				(thickness 0.1905)
+				(bold yes)
+			)
+			(justify left mirror)
+		)
+	)
+	(gr_text "SWCLK"
+		(at 150.66 93.12 0)
+		(layer "B.SilkS")
+		(effects
+			(font
+				(size 0.762 0.762)
+				(thickness 0.1905)
+				(bold yes)
+			)
+			(justify left mirror)
+		)
+	)
+	(gr_text "GND"
+		(at 150.66 95.66 0)
+		(layer "B.SilkS")
+		(effects
+			(font
+				(size 0.762 0.762)
+				(thickness 0.1905)
+				(bold yes)
+			)
+			(justify left mirror)
+		)
+	)
